File: pcb/sensor/klima-sensor.kicad_pcb (KiCad board)
At the start: 2 copper layers, 25 x 44 mm, 9 parts, among them J1 BAT, J2 XBAT, J3 SHT31, U1 XIAO ESP32-C3

Commit message: Add M2 mounting hole to sensor PCB, mill NPTH holes in cutout
The enclosure screw passes through the sensor board and clamps it
between the back shell and the front cover. Routing is unchanged
(zero jumpers, no copper DRC errors).

Co-Authored-By: Claude Opus 5.5 <noreply@anthropic.com>
Claude-Session: https://claude.ai/code/session_01K7NEXKdzHGt5toAVue95zu
Parts:
- added H1: M2, MountingHole:MountingHole_2.2mm_M2, F.Cu at (3.60, 3.00)
